File: hardware/PCB/tstick-5gw-prosumer-pcb/tstick-5gw-prosumer-pcb.kicad_sch (KiCad schematic)
At the start: 41 parts, among them Q1 BSS138, Q2 BSS138, SW1 JSTCONNECTOR, U1 PCA9306DP

Commit message: updated kicad schematic for prsoumer t-stick board board
Parts:
- removed Q1: BSS138, Package_TO_SOT_SMD:SOT-23, symbol Transistor_FET:BSS138
- removed QWIIC1: JST-SH-1x04 1.0mm, Connector_JST:JST_SH_SM04B-SRSS-TB_1x04-1MP_P1.00mm_Horizontal, symbol Connector:Conn_01x04_Pin
- removed R3, R4: 10k, Resistor_SMD:R_0201_0603Metric, symbol Device:R_US
- added C3, C4: 1uF, Capacitor_SMD:C_0201_0603Metric, symbol Device:C
- added QWIIC1: JST-SH-1x04 1.0mm, Connector_JST:JST_SH_SM04B-SRSS-TB_1x04-1MP_P1.00mm_Horizontal, symbol Connector_Generic_MountingPin:Conn_01x04_MountingPin
- added Ud1: MAX8511EXK18+T, max8511-footprints:21-0076_X5&plus_1_MXM, symbol max8511:MAX8511EXK18+T
- BT1: symbol Device:Battery -> Connector_Generic_MountingPin:Conn_01x02_MountingPin
- FLEX1: symbol Connector_Generic:Conn_01x32 -> Connector_Generic_MountingPin:Conn_01x32_MountingPin
- FSR1: symbol Device:R_Variable_US -> Connector_Generic_MountingPin:Conn_01x02_MountingPin
- SW1: symbol Switch:SW_Push -> Connector_Generic_MountingPin:Conn_01x02_MountingPin
- TrillExtensionInput1: footprint Connector_JST:JST_SHL_SM08B-SHLS-TF_1x08-1MP_P1.00mm_Horizontal -> Connector_JST:JST_SH_SM04B-SRSS-TB_1x04-1MP_P1.00mm_Horizontal; symbol Connector_Generic:Conn_01x08 -> Connector_Generic_MountingPin:Conn_01x04_MountingPin; Description Value Pkg Connector Header Surface Mount, Right Angle 8 position 0.03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 -> Connector Header Surface Mount, Right Angle 4 position 0.03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; Digikey Part # 455-3960-1-ND -> 455-1804-1-ND; Mfg Part # SM08B-SHLS-TF -> SM04B-SRSS-TB(LF)(SN)
Connections:
- net FG_INT is gone; now on net IO4: FG1.8 (ALRT)
- net +1V8: now also C3.1, Ud1.5 (OUT); no longer C2.1, FG1.7 (REG)
- net +3V3: now also C4.1, QWIIC1.2 (Pin_2), Ud1.1 (IN), Ud1.3 (*SHDN); no longer TrillExtensionInput1.2 (Pin_2)
- net -BATT: now also BT1.MP (MountPin)
- net GND: now also FLEX1.MP (MountPin), FSR1.MP (MountPin), SW1.MP (MountPin), TrillExtensionInput1.MP (MountPin), C3.2, C4.2, QWIIC1.1 (Pin_1), QWIIC1.MP (MountPin), Ud1.2 (GND); no longer TrillExtensionInput1.1 (Pin_1)
- net IO14: now also TrillExtensionInput1.4 (Pin_4); no longer TrillExtensionInput1.8 (Pin_8)
- net IO25: now also TrillExtensionInput1.3 (Pin_3); no longer TrillExtensionInput1.7 (Pin_7)
- net IO26: now also TrillExtensionInput1.2 (Pin_2); no longer TrillExtensionInput1.6 (Pin_6)
- net IO5/SS: now also TrillExtensionInput1.1 (Pin_1); no longer TrillExtensionInput1.5 (Pin_5)
- net LV_SCL: no longer FG1.3 (SCL)
- net LV_SDA: no longer FG1.4 (SDA)
- net SCL: now also FG1.3 (SCL), QWIIC1.4 (Pin_4); no longer TrillExtensionInput1.4 (Pin_4)
- net SDA: now also FG1.4 (SDA), QWIIC1.3 (Pin_3); no longer TrillExtensionInput1.3 (Pin_3)
- new net REG: C2.1, FG1.7 (REG)
- no-connect marks 7 -> 8
Other:
- note added: "4 pin JST-SH connector to daisy chain additonal touch boards"
- note added: "We have to shift the logic level from 1.8V to 3.3V to use with the TinyPico for the IMU"
- note removed: "1.8V comes from the Fuel Gauge Regulator"
- note removed: "8pin JST-SH connector to daisy chain additonal touch boards"
- note removed: "We have to shift the logic level from 1.8V to 3.3V to use with the TinyPico for both the fuel gauge and IMU"
- moved on the sheet: IMU1, Q2, R11, R12
