File: hardware/PCB/tstick-trill-touch-board/tstick-touch-board-paper/tstick-touch-board-paper.kicad_sch (KiCad schematic)
At the start: 12 parts, among them J1 Conn_01x30

Commit message: cleaned up the pcb designs for the touch extension boards, created BOM and gerber files for fabrication and assembly
Parts:
- removed TrillExtensionInput1, TrillExtensionOutput2: Conn_01x08, Connector_JST:JST_SHL_SM08B-SHLS-TF_1x08-1MP_P1.00mm_Horizontal, symbol Connector_Generic:Conn_01x08
- added I2C1, I2C2, INT1, INT2: Conn_01x04, Connector_JST:JST_SH_SM04B-SRSS-TB_1x04-1MP_P1.00mm_Horizontal, symbol Connector_Generic_MountingPin:Conn_01x04_MountingPin
- J1: now left out of the parts list
Connections:
- net +3V3: now also I2C1.2 (Pin_2), I2C2.2 (Pin_2)
- net EVT1: now also INT1.1 (Pin_1), INT2.1 (Pin_1)
- net EVT2: now also INT1.2 (Pin_2), INT2.2 (Pin_2)
- net EVT3: now also INT1.3 (Pin_3), INT2.3 (Pin_3)
- net EVT4: now also INT1.4 (Pin_4), INT2.4 (Pin_4)
- net GND: now also I2C1.1 (Pin_1), I2C1.MP (MountPin), I2C2.1 (Pin_1), I2C2.MP (MountPin), INT1.MP (MountPin), INT2.MP (MountPin)
- net SCL: now also I2C1.4 (Pin_4), I2C2.4 (Pin_4)
- net SDA: now also I2C1.3 (Pin_3), I2C2.3 (Pin_3)
Other:
- note added: "I2C Qwiic Connectors"
- note added: "Interrupt Connectors"
- note removed: "Input cable from other touch boards"
- company: (none) -> Input Devices and Musical Interaction Lab
- title: (none) -> T-Stick Trill Touch Board vPaper
- moved on the sheet: H1, H2, J1, JP1, JP2, JP3, JP4, TOUCH1, TOUCH2, TRILL1
