File: hardware/PCB/tstick-5gw-pro-pcb/_autosave-tstick-5gw-pro-pcb.kicad_sch (KiCad schematic)
At the start: 57 parts, among them J1 USB_C_Receptacle_USB2.0, J2 GPIO2, J3 GPIO1, Q1 MBT3904DW1, Q2 20V/4.2A/52mOhm/1.4W, Q3 BSS138, SW1 JST-SH-1.00mm 1x2, SW2 PTS810 SJM Switch, SW3 PTS810 SJM Switch, U1 XC6222B331MR-G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

Commit message: finished v2 of layout
Parts:
- PWLED1: footprint neopixel:2659 -> 2659:2659
Changed lines of the file:
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@@
       (effects (font (size 1.27 1.27)))
     )
-    (property "Footprint" "neopixel:2659" (at 299.72 156.21 0)
+    (property "Footprint" "2659:2659" (at 299.72 156.21 0)
       (effects (font (size 1.27 1.27)) (justify bottom) hide)
     )
