File: hardware/PCB/tstick-touch-board-CraftV2 - Copper/tstick-touch-board-CraftV2-Copper.kicad_pcb (KiCad board)
At the start: 2 copper layers, 85.6 x 31.8 mm, 12 parts, among them J1 Conn_01x32, U1 Trill_Craft

Commit message: fixed errors in schematic, added support for V1 Trill boards in v2 board design, changed headers to vertical headers in touch board
Parts:
- J1: value Conn_01x32 -> Conn_01x30; footprint ffc_footprints:CON_541323262_MOL -> touch-sensors:tstick-buttons
- moved I2C1 148.6 mm to (281.3, 128.4)
- moved INT1 148.6 mm to (281.3, 120.6)
- moved H2 133.5 mm to (293.6, 122.7)
- moved J1 130.3 mm to (78.3, 145.5)
- moved I2C2 125.6 mm to (336.8, 129.0)
- moved INT2 125.6 mm to (336.8, 121.2)
- moved H1 113.5 mm to (311.6, 121.1)
- moved U1 42.8 mm to (200.1, 126.2)
- moved JP1 42.7 mm to (164.9, 119.8)
- moved JP2 42.7 mm to (164.9, 122.3)
- moved JP3 42.7 mm to (164.9, 124.8)
- moved JP4 42.7 mm to (164.9, 127.4)
Connections:
- J1 pad 1: GND -> /TOUCH0
- J1 pad 10: /TOUCH8 -> /TOUCH9
- J1 pad 11: /TOUCH9 -> /TOUCH10
- J1 pad 12: /TOUCH10 -> /TOUCH11
- J1 pad 13: /TOUCH11 -> /TOUCH12
- J1 pad 14: /TOUCH12 -> /TOUCH13
- J1 pad 15: /TOUCH13 -> /TOUCH14
- J1 pad 16: /TOUCH14 -> /TOUCH29
- J1 pad 17: /TOUCH15 -> /TOUCH28
- J1 pad 18: /TOUCH16 -> /TOUCH27
- J1 pad 19: /TOUCH17 -> /TOUCH26
- J1 pad 2: /TOUCH0 -> /TOUCH1
- J1 pad 20: /TOUCH18 -> /TOUCH25
- J1 pad 21: /TOUCH19 -> /TOUCH24
- J1 pad 22: /TOUCH20 -> /TOUCH23
- J1 pad 23: /TOUCH21 -> /TOUCH22
- J1 pad 24: /TOUCH22 -> /TOUCH21
- J1 pad 25: /TOUCH23 -> /TOUCH20
- J1 pad 26: /TOUCH24 -> /TOUCH19
- J1 pad 27: /TOUCH25 -> /TOUCH18
- J1 pad 28: /TOUCH26 -> /TOUCH17
- J1 pad 29: /TOUCH27 -> /TOUCH16
- J1 pad 3: /TOUCH1 -> /TOUCH2
- J1 pad 30: /TOUCH28 -> /TOUCH15
- J1 pad 4: /TOUCH2 -> /TOUCH3
- J1 pad 5: /TOUCH3 -> /TOUCH4
- J1 pad 6: /TOUCH4 -> /TOUCH5
- J1 pad 7: /TOUCH5 -> /TOUCH6
- J1 pad 8: /TOUCH6 -> /TOUCH7
- J1 pad 9: /TOUCH7 -> /TOUCH8
Routing:
- net /TOUCH15: track 24.8 -> 167.5 mm, vias 1 -> 0
- net /TOUCH16: track 26.9 -> 159.3 mm, vias 1 -> 0
- net /TOUCH17: track 28.7 -> 154.7 mm, vias 1 -> 0
- net /TOUCH18: track 31.5 -> 143.1 mm, vias 1 -> 0
- net /TOUCH19: track 34.2 -> 136.0 mm, vias 1 -> 0
- net /EVT4: track 94.8 -> 0.00 mm, vias 2 -> 0
- net /EVT3: track 92.4 -> 0.00 mm, vias 2 -> 0
- net /TOUCH20: track 37.0 -> 128.4 mm, vias 1 -> 0
- net /EVT2: track 90.0 -> 0.00 mm, vias 2 -> 0
- net /EVT1: track 84.9 -> 0.00 mm
- net /TOUCH21: track 40.4 -> 121.1 mm, vias 1 -> 0
- net +3V3: track 77.7 -> 0.00 mm, vias 2 -> 0
- net /SCL: track 77.5 -> 0.00 mm, vias 2 -> 0
- net /SDA: track 75.8 -> 0.00 mm, vias 2 -> 0
- net /TOUCH22: track 43.4 -> 115.3 mm, vias 1 -> 0
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Other:
- board outline removed
