File: hardware/PCB/tstick-touch-board-RigidFlex/tstick-touch-board-RigidFlex.kicad_pcb (KiCad board)
At the start: 2 copper layers, 302.3 x 68.6 mm, 12 parts, among them J1 Conn_01x30, U1 Trill_Craft

Commit message: added stiffener location details to pcb
Other:
- board text added: "Stiffener: FR4 Side: BOTTOM Location: Shown by rectangle in User Comments Layer Thickness: 0.2mm L = 82.55mm W = 31.75mm"
Changed lines of the file:
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@@
     (effects (font (size 5 5) (thickness 1) bold) (justify left bottom))
+  )
+  (gr_text "Stiffener: FR4\nSide: BOTTOM\nLocation: Shown by rectangle in User Comments Layer\nThickness: 0.2mm\nL = 82.55mm\nW = 31.75mm" (at 223.25 74.425) (layer "Cmts.User")
+    (effects (font (size 1 1) (thickness 0.15)) (justify left bottom))
   )
   (dimension (type aligned) (layer "Cmts.User")
