File: hardware/PCB/tstick-5gw-pro-USB-V2-pcb/tstick-5gw-pro-USB-V2-pcb.kicad_sch (KiCad schematic)
At the start: 66 parts, among them J1 USB_C_Receptacle_USB2.0, Q1 BSS138, Q2 BSS138, Q3 BSS138, SW1 JST-SH-1.00mm 1x2, SW2 PTS810 SJM Switch, SW3 PTS810 SJM Switch, U1 USBLC6-2P6, U2 MCP73871, U3 NCP167AMX330TBG, U4 NCP167AMX180TBG

Commit message: updated BOM, cleaned up esp32 and touch board schematic (removed unused fields)
Parts:
- removed QWIIC1, TrillExtensionInput1: JST-SH-1x04 1.0mm, Connector_JST:JST_SH_BM04B-SRSS-TB_1x04-1MP_P1.00mm_Vertical, symbol Connector_Generic_MountingPin:Conn_01x04_MountingPin
- removed SW1: JST-SH-1.00mm 1x2, Connector_JST:JST_SH_BM02B-SRSS-TB_1x02-1MP_P1.00mm_Vertical, symbol Connector_Generic_MountingPin:Conn_01x02_MountingPin
- added ANG2: JST-SH-1.00mm 1x2, Connector_JST:JST_SH_BM02B-SRSS-TB_1x02-1MP_P1.00mm_Vertical, symbol Connector_Generic_MountingPin:Conn_01x02_MountingPin
- added TOUCH1, TOUCH2: JST-SH-1x04 1.0mm, Connector_JST:JST_SH_BM04B-SRSS-TB_1x04-1MP_P1.00mm_Vertical, symbol Connector_Generic_MountingPin:Conn_01x04_MountingPin
- ANG1: renamed from FSR1; Digikey Part # 455-1788-1-ND -> (none); Manufacturer (none) -> JST Sales America Inc.; mpn (none) -> BM02B-SRSS-TB
- BT1: Digikey Part # 455-S2B-PH-SM4-TBTR-ND -> (none); Manufacturer (none) -> JST Sales America Inc.; Mfg Part # B2B-PH-SM4-TBT -> B2B-PH-SM4-TB; mpn (none) -> B2B-PH-SM4-TBT
- C1: Digikey Part # 1276-1115-2-ND -> (none); Manufacturer (none) -> Samsung Electro-Mechanics; mpn (none) -> CL03A104KP3NNNC
- C10, C11, C12, C4, C5, C9: Digikey Part # 1276-1323-1-ND -> (none); Manufacturer (none) -> Samsung Electro-Mechanics; mpn (none) -> CL03A105KQ3CSNC
- C13, C15, C6, C7: Digikey Part # 1276-1115-1-ND -> (none); Manufacturer (none) -> Samsung Electro-Mechanics; mpn (none) -> CL03A104KP3NNNC
- C14: Manufacturer (none) -> Samsung Electro-Mechanics; mpn (none) -> CL10A106KQ8NNNC
- C2: Digikey Part # 1276-1337-1-ND -> (none); Manufacturer (none) -> Samsung Electro-Mechanics; mpn (none) -> CL03A474KQ3NNNC
- C3, C8: Digikey Part # 1276-CL03A475MQ5C65CCT-ND -> (none); Manufacturer (none) -> Samsung Electro-Mechanics; mpn (none) -> CL03A475MQ5C65C
- CHARGLED1, CHARGLED2, CHARGLED3: Manufacturer (none) -> Kingbright; mpn (none) -> APHHS1005SURCK
- FG1: Digikey Part # MAX17055ETB+TCT-ND -> (none); Manufacturer (none) -> Analog Devices Inc./Maxim Integrated; mpn (none) -> MAX17055ETB+T
- IMU1: Digikey Part # 1428-1123-1-ND -> (none); Manufacturer (none) -> TDK InvenSense; mpn (none) -> ICM-20948
- J1: Digikey Part # 2073-USB4105-GF-ACT-ND -> (none); Manufacturer (none) -> GCT; mpn (none) -> USB4105-GF-A
- MCU1: Digikey Part # 1965-ESP32-S3-WROOM-2-N32R8VCT-ND -> (none); Manufacturer (none) -> Espressif Systems; mpn (none) -> ESP32-S3-WROOM-2-N32R8V
- PWLED1: Check_prices https://www.snapeda.com/parts/2659/Adafruit+Industries+LLC/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 -> (none); Digikey Part # 1528-4492-ND -> (none); MANUFACTURER Adafruit Industries LLC -> (none); MF Adafruit Industries -> (none); MP 2659 -> (none); Manufacturer (none) -> Adafruit Industries LLC; PARTREV 01 -> (none); Package None -> (none); STANDARD Manufacturer Recommendations -> (none); SnapEDA_Link https://www.snapeda.com/parts/2659/Adafruit+Industries+LLC/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 -> (none); mpn (none) -> 4492
- Q1, Q2, Q3: Digikey Part # 4530-BSS138CT-ND -> (none); Manufacturer (none) -> ANBON SEMICONDUCTOR (INT'L) LIMITED; mpn (none) -> BSS138
- R1, R22, R24, R3: Digikey Part # P122413CT-ND -> (none); Manufacturer (none) -> Panasonic Electronic Components; mpn (none) -> ERJ-1GNF1001C
- R12, R5: Digikey Part # P122414CT-ND -> (none); Manufacturer (none) -> Panasonic Electronic Components; mpn (none) -> ERJ-1GNF1002C
- R14, R15, R16, R19, R21, R23: Digikey Part # P122832CT-ND -> (none); Manufacturer (none) -> Panasonic Electronic Components; mpn (none) -> ERJ-1GNF2201C
- R17: Manufacturer (none) -> Panasonic Electronic Components; mpn (none) -> ERJ-1GNF2492C
- R18: Manufacturer (none) -> Panasonic Electronic Components; mpn (none) -> ERJ-1GNF3303C
- R2: Digikey Part # 273-LVK12R010CERCT-ND -> (none); Manufacturer (none) -> Ohmite; mpn (none) -> LVK12R010CER
- R20: Manufacturer (none) -> Panasonic Electronic Components; mpn (none) -> ERJ-1GNF2001C
- R4: Manufacturer (none) -> Panasonic Electronic Components; mpn (none) -> ERJ-1GNF1103C
- R6, R7: Digikey Part # P123340CT-ND -> (none); Manufacturer (none) -> Panasonic Electronic Components; mpn (none) -> ERJ-1GNJ512C
- R8: Digikey Part # P122911CT-ND -> (none); Manufacturer (none) -> Panasonic Electronic Components; mpn (none) -> ERJ-1GNF3000C
- SW1: renamed from SW2; Digikey Part # CKN10502CT-ND -> (none); Manufacturer (none) -> C&K; mpn (none) -> PTS810 SJM 250 SMTR LFS
- SW2: renamed from SW3; Digikey Part # CKN10502CT-ND -> (none); Manufacturer (none) -> C&K; mpn (none) -> PTS810 SJM 250 SMTR LFS
- TH1, TH2: Digikey Part # P124053CT-ND -> (none); Manufacturer (none) -> Panasonic Electronic Components; mpn (none) -> ERT-JZEG103FA
- U1: Manufacturer (none) -> STMicroelectronics; mpn (none) -> USBLC6-2P6
- U2: Manufacturer (none) -> Microchip Technology; mpn (none) -> MCP73871-2CCI/ML
- U3: Manufacturer (none) -> onsemi; mpn (none) -> NCP167AMX330TBG
- U4: Manufacturer (none) -> onsemi; mpn (none) -> NCP167AMX180TBG
Connections:
- net +3V3: now also BOARDLAYOUT1.21 (3v3), TOUCH1.2 (Pin_2); no longer BOARDLAYOUT1.20 (3v3)
- net CIPO: now also BOARDLAYOUT1.17 (CIPO); no longer BOARDLAYOUT1.16 (CIPO)
- net COPI: now also BOARDLAYOUT1.15 (COPI); no longer BOARDLAYOUT1.14 (COPI)
- net EN: now also BOARDLAYOUT1.9 (EN); no longer BOARDLAYOUT1.8 (EN)
- net GND: now also BOARDLAYOUT1.10 (GND), BOARDLAYOUT1.20 (GND), ANG2.2 (Pin_2), ANG2.MP (MountPin), TOUCH1.1 (Pin_1), TOUCH1.MP (MountPin), TOUCH2.MP (MountPin); no longer BOARDLAYOUT1.19 (GND), BOARDLAYOUT1.9 (GND)
- net IO1: now also BOARDLAYOUT1.11 (IO01); no longer BOARDLAYOUT1.10 (IO01)
- net IO2: now also BOARDLAYOUT1.12 (IO02); no longer BOARDLAYOUT1.11 (IO02)
- net IO4: now also BOARDLAYOUT1.13 (IO04), TOUCH2.1 (Pin_1); no longer BOARDLAYOUT1.12 (IO04)
- net IO46: now also BOARDLAYOUT1.6 (LEDPOWER)
- net IO5: now also BOARDLAYOUT1.14 (IO05), TOUCH2.2 (Pin_2); no longer BOARDLAYOUT1.13 (IO05)
- net IO6: now also BOARDLAYOUT1.8 (IO06), TOUCH2.3 (Pin_3); no longer BOARDLAYOUT1.7 (IO06)
- net IO7: now also BOARDLAYOUT1.7 (IO07), TOUCH2.4 (Pin_4); no longer BOARDLAYOUT1.6 (IO07)
- net IO9: now also ANG2.1 (Pin_1)
- net SCK: now also BOARDLAYOUT1.16 (SCK); no longer BOARDLAYOUT1.15 (SCK)
- net SCL: now also BOARDLAYOUT1.19 (SCL), TOUCH1.4 (Pin_4); no longer BOARDLAYOUT1.18 (SCL)
- net SDA: now also BOARDLAYOUT1.18 (SDA), TOUCH1.3 (Pin_3); no longer BOARDLAYOUT1.17 (SDA)
- net VUSB: now also BOARDLAYOUT1.22 (5v); no longer BOARDLAYOUT1.21 (5v)
Other:
- note added: "4 pin JST-SH connector to daisy chain touch board interrupts, alternatively can connect up to 4 sensor pads for touch sensing on ESP32"
- note added: "BOARD LAYOUT"
- note added: "BOOT BUTTON"
- note added: "BUTTON/ANALOG CONNECTOR"
- note added: "CHARGER CONFIGURATION"
- note added: "CHARGING STATUS LEDS"
- note added: "Charger+PowerPath MCP73871"
- note added: "Comms - SDA: IO12 - SCL: IO11 - USBD+: IO20 - USBD-: IO19 Peripherals - FSR: IO9 - Button: IO3 - UART TX: IO43 - UART RX: IO44 - Status LED: IO10 - Status LED Power: I046 - Extra LEDs: I08 Interrupts - IMU Interrupt: IO21 - Fuel Gauge Interrupt: IO17 - Touch Interrupt 1: IO1 - Touch Interrupt 2: IO2 - Touch Interrupt 3: IO3 - Touch Interrupt 4: IO4"
- note added: "ESP32 WROOM 2 MODULE N32R8V"
- note added: "Extra neopixel LEDs can be connected to I08"
- note added: "FSR CONNECTOR"
- note added: "FUEL GAUGE"
- note added: "GPIO/TOUCH CONNECTOR"
- note added: "I2C OUT"
- note added: "IMU"
- note added: "LIPO/LI-ION CONNECTOR"
- note added: "LVL SHIFTING"
- note added: "MOUNTING HOLES (M3)"
- note added: "RESET BUTTON"
- note added: "STATUS LED"
- note added: "SYSTEM REGULATORS"
- note added: "Table 5.1 in MCP73871 Datasheet shows table for status outputs"
- note added: "Touch Board Interrupt Pins - EVT1: IO7 - EVT2: IO6 - EVT3: IO5 - EVT4: IO4"
- note added: "USB C CONNECTOR"
- note removed: "4 pin JST-SH connector to daisy chain additonal touch boards"
- note removed: "Comms - SDA: IO12 - SCL: IO11 - USBD+: IO20 - USBD-: IO19 Peripherals - FSR: IO9 - Button: IO3 - UART TX: IO43 - UART RX: IO44 - Status LED: IO10 - Status LED Power: I046 - Extra LEDs: I08 Interrupts - IMU Interrupt: IO21 - Fuel Gauge Interrupt: IO17 - Touch Interrupt 1: IO42 - Touch Interrupt 2: IO41 - Touch Interrupt 3: IO40 - Touch Interrupt 4: IO39"
- note removed: "Touch Board Interrupt Pins - EVT1: IO42 - EVT2: IO41 - EVT3: IO40 - EVT4: IO39"
- note removed: "Vertical JST Connector Footprint is used for easy removal"
- moved on the sheet: ANG1, BT1, PWLED1, R1, R8, SW1, SW2
