File: hardware/PCB/tstick-touch-board-CraftV2/tstick-touch-board-CraftV2.kicad_sch (KiCad schematic)
At the start: 12 parts, among them J1 Conn_01x32, U1 Trill_Craft

Commit message: fixed errors in schematic, added support for V1 Trill boards in v2 board design, changed headers to vertical headers in touch board
Parts:
- I2C1, I2C2, INT1, INT2: footprint Connector_JST:JST_SH_SM04B-SRSS-TB_1x04-1MP_P1.00mm_Horizontal -> JST Connectors:JST_SH_BM04B-SRSS-TB_1x04-1MP_P1.00mm_Vertical; Digikey Part # 455-SM04B-SRSS-TBCT-ND -> (none); Mfg Part # SM04B-SRSS-TB -> BM04B-SRSS-TB
Connections:
- net EVT1: now also INT1.4 (Pin_4), INT2.4 (Pin_4); no longer INT1.1 (Pin_1), INT2.1 (Pin_1)
- net EVT2: now also INT1.3 (Pin_3), INT2.3 (Pin_3); no longer INT1.2 (Pin_2), INT2.2 (Pin_2)
- net EVT3: now also INT1.2 (Pin_2), INT2.2 (Pin_2); no longer INT1.3 (Pin_3), INT2.3 (Pin_3)
- net EVT4: now also INT1.1 (Pin_1), INT2.1 (Pin_1); no longer INT1.4 (Pin_4), INT2.4 (Pin_4)
Other:
- moved on the sheet: I2C1, I2C2

Commit message: updated BOM, cleaned up esp32 and touch board schematic (removed unused fields)
Parts:
- I2C1, I2C2, INT1, INT2: Manufacturer (none) -> JST Sales America Inc.
- J1: Digikey Part # 900-0541323262CT-ND -> (none); Manufacturer (none) -> Molex
Changed lines of the file:
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@@
       (effects (font (size 1.27 1.27)) hide)
     )
-    (property "Datasheet" "~" (at 130.81 43.18 0)
+    (property "Datasheet" "https://www.jst-mfg.com/product/pdf/eng/eSH.pdf" (at 130.81 43.18 0)
       (effects (font (size 1.27 1.27)) hide)
     )
@@
       (effects (font (size 1.27 1.27)) hide)
     )
-    (property "Alternate Part #" "" (at 130.81 43.18 0)
+    (property "Manufacturer" "JST Sales America Inc." (at 130.81 43.18 0)
       (effects (font (size 1.27 1.27)) hide)
     )
@@
       (effects (font (size 1.27 1.27)) hide)
     )
+    (property "Manufacturer" "" (at 36.83 165.1 0)
+      (effects (font (size 1.27 1.27)) hide)
+    )
     (instances
       (project "tstick-touch-board"
@@
       (effects (font (size 1.27 1.27)) hide)
     )
+    (property "Manufacturer" "" (at 152.4 118.11 0)
+      (effects (font (size 1.27 1.27)) hide)
+    )
     (pin "1")
     (pin "2")
@@
       (effects (font (size 1.27 1.27)) hide)
     )
-    (property "Datasheet" "~" (at 162.56 43.18 0)
+    (property "Datasheet" "https://www.jst-mfg.com/product/pdf/eng/eSH.pdf" (at 162.56 43.18 0)
       (effects (font (size 1.27 1.27)) hide)
     )
@@
       (effects (font (size 1.27 1.27)) hide)
     )
-    (property "Alternate Part #" "" (at 162.56 43.18 0)
+    (property "Manufacturer" "JST Sales America Inc." (at 162.56 43.18 0)
       (effects (font (size 1.27 1.27)) hide)
     )
@@
       (effects (font (size 1.27 1.27)) hide)
     )
+    (property "Manufacturer" "" (at 152.4 149.86 0)
+      (effects (font (size 1.27 1.27)) hide)
+    )
     (pin "1")
     (pin "2")
@@
       (effects (font (size 1.27 1.27)) hide)
     )
-    (property "Datasheet" "~" (at 251.46 67.31 0)
+    (property "Datasheet" "https://tools.molex.com/pdm_docs/ps/PS-54132-061.pdf" (at 251.46 67.31 0)
       (effects (font (size 1.27 1.27)) hide)
     )
@@
       (effects (font (size 1.27 1.27)) hide)
     )
-    (property "Digikey Part #" "900-0541323262CT-ND" (at 251.46 67.31 0)
-      (effects (font (size 1.27 1.27)) hide)
-    )
-    (property "Alternate Part #" "" (at 251.46 67.31 0)
+    (property "Manufacturer" "Molex" (at 251.46 67.31 0)
       (effects (font (size 1.27 1.27)) hide)
     )
@@
       (effects (font (size 1.27 1.27)) hide)
     )
+    (property "Manufacturer" "" (at 36.83 175.26 0)
+      (effects (font (size 1.27 1.27)) hide)
+    )
     (instances
       (project "tstick-touch-board"
@@
       (effects (font (size 1.27 1.27)) hide)
     )
-    (property "Digikey Part #" "" (at 48.26 54.61 0)
-      (effects (font (size 1.27 1.27)) hide)
-    )
-    (property "Alternate Part #" "" (at 48.26 54.61 0)
+    (property "Manufacturer" "" (at 48.26 54.61 0)
       (effects (font (size 1.27 1.27)) hide)
     )
@@
       (effects (font (size 1.27 1.27)) hide)
     )
-    (property "Datasheet" "~" (at 170.18 85.09 0)
+    (property "Datasheet" "https://www.jst-mfg.com/product/pdf/eng/eSH.pdf" (at 170.18 85.09 0)
       (effects (font (size 1.27 1.27)) hide)
     )
@@
       (effects (font (size 1.27 1.27)) hide)
     )
-    (property "Alternate Part #" "" (at 170.18 85.09 0)
+    (property "Manufacturer" "JST Sales America Inc." (at 170.18 85.09 0)
       (effects (font (size 1.27 1.27)) hide)
     )
@@
       (effects (font (size 1.27 1.27)) hide)
     )
+    (property "Manufacturer" "" (at 152.4 128.27 0)
+      (effects (font (size 1.27 1.27)) hide)
+    )
     (pin "1")
     (pin "2")
@@
       (effects (font (size 1.27 1.27)) hide)
     )
-    (property "Datasheet" "~" (at 137.16 85.09 0)
+    (property "Datasheet" "https://www.jst-mfg.com/product/pdf/eng/eSH.pdf" (at 137.16 85.09 0)
       (effects (font (size 1.27 1.27)) hide)
     )
@@
       (effects (font (size 1.27 1.27)) hide)
     )
-    (property "Alternate Part #" "" (at 137.16 85.09 0)
+    (property "Manufacturer" "JST Sales America Inc." (at 137.16 85.09 0)
       (effects (font (size 1.27 1.27)) hide)
     )
@@
       (effects (font (size 1.27 1.27)) hide)
     )
+    (property "Manufacturer" "" (at 152.4 139.7 0)
+      (effects (font (size 1.27 1.27)) hide)
+    )
