File: hardware/PCB/touch-sensor-horizontal/touch-sensor-horizontal.kicad_pcb (KiCad board)
At the start: 2 copper layers, 302.3 x 34.1 mm, 2 parts, among them J1 Conn_01x30

Commit message: updated touch sensor design to be at the end of the board, also has longer neck
Parts:
- C1, J1: moved to B.Cu
- moved C1 134.6 mm to (336.4, 118.8), turned to 180 degrees
- moved J1 2.00 mm to (56.9, 148.1)
Connections:
- C1 pad 10: /TOUCH8 -> /TOUCH21
- C1 pad 11: /TOUCH9 -> /TOUCH20
- C1 pad 12: /TOUCH10 -> /TOUCH19
- C1 pad 13: /TOUCH11 -> /TOUCH18
- C1 pad 14: /TOUCH12 -> /TOUCH17
- C1 pad 15: /TOUCH13 -> /TOUCH16
- C1 pad 16: /TOUCH14 -> /TOUCH15
- C1 pad 17: /TOUCH15 -> /TOUCH14
- C1 pad 18: /TOUCH16 -> /TOUCH13
- C1 pad 19: /TOUCH17 -> /TOUCH12
- C1 pad 2: /TOUCH0 -> /TOUCH29
- C1 pad 20: /TOUCH18 -> /TOUCH11
- C1 pad 21: /TOUCH19 -> /TOUCH10
- C1 pad 22: /TOUCH20 -> /TOUCH9
- C1 pad 23: /TOUCH21 -> /TOUCH8
- C1 pad 24: /TOUCH22 -> /TOUCH7
- C1 pad 25: /TOUCH23 -> /TOUCH6
- C1 pad 26: /TOUCH24 -> /TOUCH5
- C1 pad 27: /TOUCH25 -> /TOUCH4
- C1 pad 28: /TOUCH26 -> /TOUCH3
- C1 pad 29: /TOUCH27 -> /TOUCH2
- C1 pad 3: /TOUCH1 -> /TOUCH28
- C1 pad 30: /TOUCH28 -> /TOUCH1
- C1 pad 31: /TOUCH29 -> /TOUCH0
- C1 pad 4: /TOUCH2 -> /TOUCH27
- C1 pad 5: /TOUCH3 -> /TOUCH26
- C1 pad 6: /TOUCH4 -> /TOUCH25
- C1 pad 7: /TOUCH5 -> /TOUCH24
- C1 pad 8: /TOUCH6 -> /TOUCH23
- C1 pad 9: /TOUCH7 -> /TOUCH22
Routing:
- net /TOUCH13: track 22.4 -> 160.0 mm
- net /TOUCH12: track 31.8 -> 169.2 mm
- net /TOUCH11: track 41.2 -> 178.5 mm
- net /TOUCH10: track 50.7 -> 187.8 mm
- net /TOUCH9: track 60.1 -> 197.1 mm
- net /TOUCH8: track 69.6 -> 206.4 mm
- net /TOUCH7: track 79.1 -> 215.7 mm
- net /TOUCH5: track 97.9 -> 234.4 mm
- net /TOUCH0: track 145.3 -> 281.7 mm
- net /TOUCH2: track 126.4 -> 262.8 mm
- net /TOUCH1: track 135.9 -> 272.2 mm
- net /TOUCH4: track 107.5 -> 243.8 mm
- net /TOUCH6: track 88.6 -> 225.0 mm
- net /TOUCH3: track 117.0 -> 253.3 mm
- net /TOUCH14: track 15.3 -> 150.6 mm
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Other:
- board size 302.3 x 34.1 mm -> 302.3 x 45.7 mm
- board text added: "PI STIFFENER AREA TOP, 0.1mm"
- board text removed: "STIFFENER AREA"

Commit message: updated touch sensor design to be a slider
Parts:
- J1: value Conn_01x30 -> touch-sensor; footprint touch-sensors:tstick-buttons -> touch-sensors:tstick-slider; moved to F.Cu
- moved J1 152.1 mm to (208.9, 147.4)
Connections:
- J1 pad 1: /TOUCH0 -> GND
- J1 pad 10: /TOUCH9 -> /TOUCH8
- J1 pad 11: /TOUCH10 -> /TOUCH9
- J1 pad 12: /TOUCH11 -> /TOUCH10
- J1 pad 13: /TOUCH12 -> /TOUCH11
- J1 pad 14: /TOUCH13 -> /TOUCH12
- J1 pad 15: /TOUCH14 -> /TOUCH13
- J1 pad 16: /TOUCH15 -> /TOUCH14
- J1 pad 17: /TOUCH16 -> /TOUCH15
- J1 pad 18: /TOUCH17 -> /TOUCH16
- J1 pad 19: /TOUCH18 -> /TOUCH17
- J1 pad 2: /TOUCH1 -> /TOUCH0
- J1 pad 20: /TOUCH19 -> /TOUCH18
- J1 pad 21: /TOUCH20 -> /TOUCH19
- J1 pad 22: /TOUCH21 -> /TOUCH20
- J1 pad 23: /TOUCH22 -> /TOUCH21
- J1 pad 24: /TOUCH23 -> /TOUCH22
- J1 pad 25: /TOUCH24 -> /TOUCH23
- J1 pad 26: /TOUCH25 -> /TOUCH24
- J1 pad 27: /TOUCH26 -> /TOUCH25
- J1 pad 28: /TOUCH27 -> /TOUCH26
- J1 pad 29: /TOUCH28 -> /TOUCH27
- J1 pad 3: /TOUCH2 -> /TOUCH1
- J1 pad 30: /TOUCH29 -> /TOUCH28
- J1 pad 4: /TOUCH3 -> /TOUCH2
- J1 pad 5: /TOUCH4 -> /TOUCH3
- J1 pad 6: /TOUCH5 -> /TOUCH4
- J1 pad 7: /TOUCH6 -> /TOUCH5
- J1 pad 8: /TOUCH7 -> /TOUCH6
- J1 pad 9: /TOUCH8 -> /TOUCH7
Routing:
- net /TOUCH0: track 281.7 -> 251.6 mm
- net /TOUCH1: track 272.2 -> 243.4 mm
- net /TOUCH2: track 262.8 -> 235.5 mm
- net /TOUCH3: track 253.3 -> 227.3 mm
- net /TOUCH4: track 243.8 -> 219.4 mm
- net /TOUCH5: track 234.4 -> 211.0 mm
- net /TOUCH6: track 225.0 -> 203.2 mm
- net /TOUCH7: track 215.7 -> 195.1 mm
- net /TOUCH8: track 206.4 -> 187.6 mm
- net /TOUCH9: track 197.1 -> 179.7 mm
- net /TOUCH10: track 187.8 -> 171.5 mm
- net /TOUCH11: track 178.5 -> 164.0 mm
- net /TOUCH12: track 169.2 -> 156.0 mm
- net GND: track 16.8 -> 28.7 mm, vias 2 -> 4
- net /TOUCH13: track 160.0 -> 148.2 mm
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
Commit message: Added updated pcb manufacturing files
Routing:
- net GND: track 28.7 -> 20.2 mm
Other:
- board size 302.3 x 45.7 mm -> 284.5 x 45.7 mm
Changed lines of the file:
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@@
   (gr_rect (start 328.15 116.55) (end 344.65 120.925)
     (stroke (width 0.15) (type default)) (fill none) (layer "Cmts.User"))
-  (gr_rect (start 50.8 127) (end 353.06 167.625)
+  (gr_rect (start 66.04 127) (end 353.06 167.64)
     (stroke (width 0.15) (type default)) (fill none) (layer "Cmts.User"))
-  (gr_line (start 350.52 167.64) (end 53.34 167.64)
+  (gr_line (start 347.98 167.64) (end 68.58 167.64)
     (stroke (width 0.1) (type default)) (layer "Edge.Cuts"))
   (gr_arc (start 345.74 127) (mid 344.983396 126.686604) (end 344.67 125.93)
     (stroke (width 0.1) (type default)) (layer "Edge.Cuts"))
-  (gr_line (start 353.06 129.54) (end 353.06 165.1)
+  (gr_line (start 350.52 129.54) (end 350.52 165.1)
     (stroke (width 0.1) (type default)) (layer "Edge.Cuts"))
-  (gr_line (start 53.34 127) (end 327.1 127)
+  (gr_line (start 68.58 127) (end 327.1 127)
     (stroke (width 0.1) (type default)) (layer "Edge.Cuts"))
-  (gr_arc (start 53.34 167.64) (mid 51.543949 166.896051) (end 50.8 165.1)
+  (gr_arc (start 68.58 167.64) (mid 66.783949 166.896051) (end 66.04 165.1)
     (stroke (width 0.1) (type default)) (layer "Edge.Cuts"))
   (gr_line (start 328.17 125.93) (end 328.17 121.93)
@@
   (gr_arc (start 328.17 125.93) (mid 327.856604 126.686604) (end 327.1 127)
     (stroke (width 0.1) (type default)) (layer "Edge.Cuts"))
-  (gr_arc (start 353.06 165.1) (mid 352.316051 166.896051) (end 350.52 167.64)
+  (gr_arc (start 350.52 165.1) (mid 349.776051 166.896051) (end 347.98 167.64)
     (stroke (width 0.1) (type default)) (layer "Edge.Cuts"))
-  (gr_arc (start 50.8 129.54) (mid 51.543949 127.743949) (end 53.34 127)
+  (gr_arc (start 66.04 129.54) (mid 66.783949 127.743949) (end 68.58 127)
     (stroke (width 0.1) (type default)) (layer "Edge.Cuts"))
-  (gr_line (start 50.8 165.1) (end 50.8 129.54)
+  (gr_line (start 66.04 165.1) (end 66.04 129.54)
     (stroke (width 0.1) (type default)) (layer "Edge.Cuts"))
-  (gr_arc (start 350.52 127) (mid 352.316051 127.743949) (end 353.06 129.54)
+  (gr_arc (start 347.98 127) (mid 349.776051 127.743949) (end 350.52 129.54)
     (stroke (width 0.1) (type default)) (layer "Edge.Cuts"))
   (gr_line (start 344.67 125.93) (end 344.67 121.93)
     (stroke (width 0.1) (type default)) (layer "Edge.Cuts"))
-  (gr_line (start 345.74 127) (end 350.52 127)
+  (gr_line (start 345.74 127) (end 347.98 127)
     (stroke (width 0.1) (type default)) (layer "Edge.Cuts"))
   (gr_text "TAPE AREA \n(BOT, opposite of copper pads)" (at 154.94 149.86) (layer "Cmts.User")
@@
   (via (at 328.4443 127.0255) (size 0.8) (drill 0.4) (layers "F.Cu" "B.Cu") (net 1))
   (via (at 69.75 164.5) (size 0.8) (drill 0.4) (layers "F.Cu" "B.Cu") (net 1))
-  (via (at 345.854166 138.4) (size 0.8) (drill 0.4) (layers "F.Cu" "B.Cu") (net 1))
+  (via (at 345.5 130) (size 0.8) (drill 0.4) (layers "F.Cu" "B.Cu") (net 1))
+  (segment (start 344.17 128.67) (end 344.17 118.75) (width 0.1524) (layer "B.Cu") (net 1))
   (segment (start 328.67 126.7998) (end 328.67 118.75) (width 0.1524) (layer "B.Cu") (net 1))
-  (segment (start 344.17 136.715834) (end 344.17 118.75) (width 0.1524) (layer "B.Cu") (net 1))
   (segment (start 328.4443 127.0255) (end 328.67 126.7998) (width 0.1524) (layer "B.Cu") (net 1))
-  (segment (start 345.854166 138.4) (end 344.17 136.715834) (width 0.1524) (layer "B.Cu") (net 1))
+  (segment (start 345.5 130) (end 344.17 128.67) (width 0.1524) (layer "B.Cu") (net 1))
   (via (at 87.25 129.75) (size 0.8) (drill 0.4) (layers "F.Cu" "B.Cu") (net 2))
   (segment (start 87.25 129.75) (end 88.15 129.75) (width 0.1524) (layer "B.Cu") (net 2))

Commit message: extended length of slider back to 30cm
Parts:
- moved J1 8.08 mm to (200.9, 147.3)
Connections:
- J1 pad 1: GND -> /TOUCH0
- J1 pad 10: /TOUCH8 -> /TOUCH9
- J1 pad 11: /TOUCH9 -> /TOUCH10
- J1 pad 12: /TOUCH10 -> /TOUCH11
- J1 pad 13: /TOUCH11 -> /TOUCH12
- J1 pad 14: /TOUCH12 -> /TOUCH13
- J1 pad 15: /TOUCH13 -> /TOUCH14
- J1 pad 16: /TOUCH14 -> /TOUCH15
- J1 pad 17: /TOUCH15 -> /TOUCH16
- J1 pad 18: /TOUCH16 -> /TOUCH17
- J1 pad 19: /TOUCH17 -> /TOUCH18
- J1 pad 2: /TOUCH0 -> /TOUCH1
- J1 pad 20: /TOUCH18 -> /TOUCH19
- J1 pad 21: /TOUCH19 -> /TOUCH20
- J1 pad 22: /TOUCH20 -> /TOUCH21
- J1 pad 23: /TOUCH21 -> /TOUCH22
- J1 pad 24: /TOUCH22 -> /TOUCH23
- J1 pad 25: /TOUCH23 -> /TOUCH24
- J1 pad 26: /TOUCH24 -> /TOUCH25
- J1 pad 27: /TOUCH25 -> /TOUCH26
- J1 pad 28: /TOUCH26 -> /TOUCH27
- J1 pad 29: /TOUCH27 -> /TOUCH28
- J1 pad 3: /TOUCH1 -> /TOUCH2
- J1 pad 30: /TOUCH28 -> /TOUCH29
- J1 pad 4: /TOUCH2 -> /TOUCH3
- J1 pad 5: /TOUCH3 -> /TOUCH4
- J1 pad 6: /TOUCH4 -> /TOUCH5
- J1 pad 7: /TOUCH5 -> /TOUCH6
- J1 pad 8: /TOUCH6 -> /TOUCH7
- J1 pad 9: /TOUCH7 -> /TOUCH8
Routing:
- net /TOUCH0: track 251.6 -> 274.9 mm
- net /TOUCH1: track 243.4 -> 265.3 mm
- net /TOUCH2: track 235.5 -> 256.2 mm
- net /TOUCH3: track 227.3 -> 246.8 mm
- net /TOUCH4: track 219.4 -> 237.6 mm
- net /TOUCH5: track 211.0 -> 228.3 mm
- net /TOUCH6: track 203.2 -> 219.4 mm
- net /TOUCH7: track 195.1 -> 210.6 mm
- net /TOUCH8: track 187.6 -> 201.4 mm
- net /TOUCH9: track 179.7 -> 192.5 mm
- net /TOUCH10: track 171.5 -> 183.7 mm
- net /TOUCH11: track 164.0 -> 174.7 mm
- net /TOUCH12: track 156.0 -> 165.7 mm
- net /TOUCH13: track 148.2 -> 156.9 mm
- net /TOUCH28: track 29.0 -> 20.7 mm
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Other:
- board size 284.5 x 45.7 mm -> 299.7 x 45.7 mm
