File: hardware/PCB/touch-sensor-horizontal/touch-sensor-horizontal.kicad_pcb (KiCad board)
At the start: 2 copper layers, 299.7 x 45.7 mm, 2 parts, among them J1 touch-sensor

Commit message: Updated touch sensor design for better fit with assembly, fixed small allignment issue with touch board
Parts:
- moved J1 2.32 mm to (200.8, 145.0)
- moved C1 1.00 mm to (336.4, 117.8)
Routing:
- net /TOUCH28: track 20.7 -> 12.6 mm
- net /TOUCH27: track 31.6 -> 24.8 mm
- net /TOUCH26: track 40.8 -> 34.2 mm
- net /TOUCH25: track 49.9 -> 44.1 mm
- net /TOUCH29: track 11.5 -> 16.4 mm
- net /TOUCH24: track 58.7 -> 53.8 mm
- net /TOUCH23: track 67.6 -> 63.3 mm
- net /TOUCH22: track 76.6 -> 72.6 mm
- net /TOUCH21: track 85.4 -> 81.9 mm
- net /TOUCH20: track 94.3 -> 91.1 mm
- net GND: track 16.7 -> 19.8 mm
- net /TOUCH19: track 103.3 -> 100.3 mm
- net /TOUCH18: track 112.4 -> 109.5 mm
- net /TOUCH1: track 265.3 -> 267.9 mm
- net /TOUCH17: track 121.3 -> 118.8 mm
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Other:
- board size 299.7 x 45.7 mm -> 306.1 x 41.6 mm

Commit message: updated touch sensor files
Other:
- board text added: "TAPE AREA (BOT)"
- board text removed: "TAPE AREA (BOT, opposite of copper pads)"
Changed lines of the file:
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@@
   (gr_line (start 345.74 127) (end 354.33 127)
     (stroke (width 0.1) (type default)) (layer "Edge.Cuts"))
-  (gr_text "TAPE AREA \n(BOT, opposite of copper pads)" (at 153.67 156.21) (layer "Cmts.User")
+  (gr_text "TAPE AREA \n(BOT)" (at 153.67 156.21) (layer "Cmts.User")
     (effects (font (size 5 5) (thickness 1) bold) (justify left bottom))
   )
