File: hardware/PCB/touch-sensor-horizontal/touch-sensor-horizontal.kicad_sch (KiCad schematic)
At the start: 2 parts, among them J1 Conn_01x30

Commit message: add updated project files
Parts:
- J1: value Conn_01x30 -> touch-sensor; footprint touch-sensors:tstick-buttons -> touch-sensors:tstick-slider
Connections:
- net TOUCH0: now also C1.31 (Sense30); no longer C1.2 (Sense1)
- net TOUCH1: now also C1.30 (Sense29); no longer C1.3 (Sense2)
- net TOUCH10: now also C1.21 (Sense20); no longer C1.12 (Sense11)
- net TOUCH11: now also C1.20 (Sense19); no longer C1.13 (Sense12)
- net TOUCH12: now also C1.19 (Sense18); no longer C1.14 (Sense13)
- net TOUCH13: now also C1.18 (Sense17); no longer C1.15 (Sense14)
- net TOUCH14: now also C1.17 (Sense16); no longer C1.16 (Sense15)
- net TOUCH15: now also C1.16 (Sense15); no longer C1.17 (Sense16)
- net TOUCH16: now also C1.15 (Sense14); no longer C1.18 (Sense17)
- net TOUCH17: now also C1.14 (Sense13); no longer C1.19 (Sense18)
- net TOUCH18: now also C1.13 (Sense12); no longer C1.20 (Sense19)
- net TOUCH19: now also C1.12 (Sense11); no longer C1.21 (Sense20)
- net TOUCH2: now also C1.29 (Sense28); no longer C1.4 (Sense3)
- net TOUCH20: now also C1.11 (Sense10); no longer C1.22 (Sense21)
- net TOUCH21: now also C1.10 (Sense9); no longer C1.23 (Sense22)
- net TOUCH22: now also C1.9 (Sense8); no longer C1.24 (Sense23)
- net TOUCH23: now also C1.8 (Sense7); no longer C1.25 (Sense24)
- net TOUCH24: now also C1.7 (Sense6); no longer C1.26 (Sense25)
- net TOUCH25: now also C1.6 (Sense5); no longer C1.27 (Sense26)
- net TOUCH26: now also C1.5 (Sense4); no longer C1.28 (Sense27)
- net TOUCH27: now also C1.4 (Sense3); no longer C1.29 (Sense28)
- net TOUCH28: now also C1.3 (Sense2); no longer C1.30 (Sense29)
- net TOUCH29: now also C1.2 (Sense1); no longer C1.31 (Sense30)
- net TOUCH3: now also C1.28 (Sense27); no longer C1.5 (Sense4)
- net TOUCH4: now also C1.27 (Sense26); no longer C1.6 (Sense5)
- net TOUCH5: now also C1.26 (Sense25); no longer C1.7 (Sense6)
- net TOUCH6: now also C1.25 (Sense24); no longer C1.8 (Sense7)
- net TOUCH7: now also C1.24 (Sense23); no longer C1.9 (Sense8)
- net TOUCH8: now also C1.23 (Sense22); no longer C1.10 (Sense9)
- net TOUCH9: now also C1.22 (Sense21); no longer C1.11 (Sense10)
