File: hardware/PCB/enchanti-touch-board/enchanti-touch-board.kicad_sch (KiCad schematic)
At the start: 91 parts, among them J2 Progamming Header, U1 CY8C4149AZI-S598

Commit message: rename PCB files to enchantiS3, exposed SPI pins for touch board
Renamed ESP32 board PCB files to EnchantiS3
Exposed SPI pins for enchanti touch board
Changed Aux touch board connector to two 4 pin JST SM connectors
Updated Enchanti touch board BOM an manufacturing files
Parts:
- removed GPIO3: SPI, Connector_JST:JST_SH_BM08B-SRSS-TB_1x08-1MP_P1.00mm_Vertical, symbol Connector_Generic_MountingPin:Conn_01x08_MountingPin
- added GPIO2: I2C, JST-footprints:JST_SH_BM04B-SRSS-TB_1x04-1MP_P1.00mm_Vertical, symbol Connector_Generic_MountingPin:Conn_01x04_MountingPin
- added GPIO4: SPI2, JST-footprints:JST_SH_BM04B-SRSS-TB_1x04-1MP_P1.00mm_Vertical, symbol Connector_Generic_MountingPin:Conn_01x04_MountingPin
- GPIO3: renamed from GPIO2; value INTERRUPT -> SPI1
- GPIO5: renamed from GPIO4; symbol Connector_Generic:Conn_01x04 -> Connector_Generic:Conn_01x02
Connections:
- net MSC046 is gone; now on net CMOD00: U1.45 (P4.2)
- net MSC047 is gone; now on net CMOD01: U1.46 (P4.3)
- net +3V3: now also GPIO2.2 (Pin_2)
- net CMOD00: no longer U1.43 (P4.0)
- net CMOD01: no longer U1.44 (P4.1)
- net EVT_AUX: no longer GPIO3.2 (Pin_2), GPIO5.2 (Pin_2)
- net EVT_MAIN: now also GPIO5.2 (Pin_2); no longer GPIO3.4 (Pin_4), GPIO5.4 (Pin_4)
- net GND: now also GPIO2.1 (Pin_1), GPIO2.MP (MountPin), GPIO4.MP (MountPin)
- net POLL_AUX: no longer GPIO3.1 (Pin_1), GPIO5.1 (Pin_1)
- net POLL_MAIN: now also GPIO5.1 (Pin_1); no longer GPIO3.3 (Pin_3), GPIO5.3 (Pin_3)
- net CS renamed CS_AUX
- net CS_AUX: now also GPIO4.4 (Pin_4)
- net MISO renamed CIPO_AUX
- net CIPO_AUX: now also GPIO4.1 (Pin_1)
- net MOSI renamed COPI_AUX
- net COPI_AUX: now also GPIO4.3 (Pin_3)
- net MSC043: no longer names the net of U1.41 (P11.5)
- net MSC048 renamed COPI_MAIN
- net COPI_MAIN: now also GPIO3.3 (Pin_3)
- net MSC049 renamed CIPO_MAIN
- net CIPO_MAIN: now also GPIO3.1 (Pin_1)
- net MSC050 renamed SCLK_MAIN
- net SCLK_MAIN: now also GPIO3.2 (Pin_2)
- net MSC051 renamed CS_MAIN
- net CS_MAIN: now also GPIO3.4 (Pin_4)
- net P30: no longer names the net of U1.27 (P3.0)
- net P30: no longer R1.1
- net P31: no longer names the net of U1.28 (P3.1)
- net P31: no longer R2.1
- net SPICLK renamed SCLK_AUX
- net SCLK_AUX: now also GPIO4.2 (Pin_2)
- new net P40: R1.1, U1.43 (P4.0)
- new net P41: R2.1, U1.44 (P4.1)
- no-connect marks 2 -> 7
Other:
- note added: "4 Pin header for SPI"
- note added: "Connect to Extra Touch board"
- note added: "Connect to MCU"
- note added: "Pads for checking evts on oscilloscope/ other MCU"
- note added: "Programming Header for 10 pin Ribbon Cable"
- note removed: "4 Pin header for testing scan speeds, poll rates and interrupts"
- note removed: "8 pin header for SPI For external boards"
- note removed: "Pads for checking evts on oscilloscope"
- note removed: "Programming Header for CY8CKIT-005-A Ribbon Cable"
- note removed: "SPI"
- note removed: "Touch IC"
- moved on the sheet: GPIO1, GPIO3, J2, R1, R2, R63, R64
