File: hardware/PCB/enchantiS3-board/enchantiS3.kicad_sch (KiCad schematic)
At the start: 71 parts, among them J1 USB_C_Receptacle_USB2.0, Q1 BSS138, Q2 BSS138, Q3 BSS138, SW1 B3U-1000P, SW2 B3U-1000P, U1 USBLC6-2P6, U2 MCP73871, U3 NCP167AMX330TBG, U4 NCP167AMX180TBG

Commit message: updated pcb files from pcb-development branch
Parts:
- removed Q1, Q2, Q3: BSS138, Package_TO_SOT_SMD:SOT-23, symbol Transistor_FET:BSS138
- removed R14, R15, R21, R23: 2k2, Resistor_SMD:R_0402_1005Metric, symbol Device:R_US
- added C16, C17, C20: 1uF, Capacitor_SMD:C_0402_1005Metric, symbol Device:C
- added C18, C21: 0.1uF, Capacitor_SMD:C_0402_1005Metric, symbol Device:C
- added SYS4: SYS, symbol power-symbols:VSYS
- added U5: NCP167AMX330TBG, XDFN4_1X1_711AJ_ONS, symbol NCP167AMX330TBG:NCP167AMX330TBG
- added U7: max3378eetd+t, 21-0137I_T1433-2_MXM, symbol MAX3378E:max3378eetd+t
- R22: value 1k -> 2k; Description Value Pkg 1 kOhms ±1% 0.1W, 1/10W Chip Resistor 0402 (1005 Metric) Au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 -> 2 kOhms ±1% 0.1W, 1/10W Chip Resistor 0402 (1005 Metric) Au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
- R24: value 1k -> 470; Description Value Pkg 1 kOhms ±1% 0.1W, 1/10W Chip Resistor 0402 (1005 Metric) Au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 -> 470 Ohms ±1% 0.1W, 1/10W Chip Resistor 0402 (1005 Metric) A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; Mfg Part # ERJ-2RKF1001X -> ERJ-2RKF4700X
- R3: value 1k -> 2k; Description Value Pkg 1 kOhms ±1% 0.1W, 1/10W Chip Resistor 0402 (1005 Metric) Au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 -> 2 kOhms ±1% 0.1W, 1/10W Chip Resistor 0402 (1005 Metric) Au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; Mfg Part # ERJ-2RKF1001X -> ERJ-2RKF2001X
Connections:
- net +1V8: now also C18.1, U7.10 (VL), U7.3 (*THREE-STATE); no longer IMU1.22 (~{CS})
- net +3V3: now also C20.1, C21.1, U7.14 (VCC); no longer TOUCH1.2 (Pin_2)
- net GND: now also C16.2, C17.2, C18.2, C20.2, C21.2, U5.2 (GND), U5.5 (GND), U7.15 (EPAD), U7.7 (GND); no longer IMU1.9 (SDO/AD0)
- net SYS: now also C17.1, SYS4.1 (SYS), U5.4 (IN); no longer U4.3 (EN)
- net IMU_INT: no longer names the net of IMU1.12 (INT1)
- net IO39 renamed COPI_AUX
- net COPI_AUX: now also U7.8 (I/O_VCC4)
- net IO40 renamed CIPO_AUX
- net CIPO_AUX: now also U7.9 (I/O_VCC3)
- net IO41 renamed CS_AUX
- net CS_AUX: now also U7.12 (I/O_VCC2)
- net IO42 renamed CLK_AUX
- net CLK_AUX: now also U7.13 (I/O_VCC1)
- net IO48 renamed LDO_EN
- net LDO_EN: now also U4.3 (EN), U5.3 (EN)
- net LV_SCL renamed CLK_1V8
- net CLK_1V8: now also U7.1 (I/O_VL1)
- net LV_SDA renamed COPI_1V8
- net COPI_1V8: now also U7.6 (I/O_VL4)
- new net +3V3_AUX: C16.1, TOUCH1.2 (Pin_2), U5.1 (OUT)
- new net CIPO_1V8: IMU1.9 (SDO/AD0), U7.5 (I/O_VL3)
- new net CS_1V8: IMU1.22 (~{CS}), U7.2 (I/O_VL2)
- no-connect marks 9 -> 10
Other:
- note added: "CHARGER CONFIG"
- note added: "Charge Termination Current 24.9koHm = 40mA charge termination"
- note added: "Charge resistor 1k = 1000mA 2k = 500mA 5k = 100mA"
- note added: "Comms - USBD+: IO20 - USBD-: IO19 - UART TX: IO43 - UART RX: IO44 I2C - SDA: IO21 - SCL: IO14 SPI - COPI: 10 - CIPO: 13 - SCLK: 12 - CS0: 11 - COPI_AUX: 39 - CIPO_AUX: 40 - CLK_AUX: 42 - CS_AUX: 41 Peripherals - LDO ENABLE: 48 - FSR: IO8 - Button: IO9 - Status LED (orange): IO16 - Status LED (blue) I015 Interrupts - Fuel Gauge Interrupt: IO17"
- note added: "ESD Protection IC"
- note added: "GPIO CONNECTORS"
- note added: "LIPO/LI-ION"
- note added: "Main 3.3V Regulator"
- note added: "Peripheral 3.3V Regulator"
- note added: "STATUS LEDS"
- note removed: "3.3V Regulator"
- note removed: "4 pin JST-SH connector to daisy chain touch board interrupts, alternatively can connect to the SPI2 controller on ESP32-S3"
- note removed: "CHARGER CONFIGURATION"
- note removed: "CHARGING STATUS LEDS"
- note removed: "Charge Limit 2kOhm = 500mA"
- note removed: "Charge Termincation Current 24.9koHm = 40mA charge termination"
- note removed: "Comms - SDA: IO21 - SCL: IO14 - USBD+: IO20 - USBD-: IO19 - COPI: 10 - CIPO: 13 - SCLK: 12 - CS0: 11 Peripherals - FSR: IO8 - Button: IO9 - UART TX: IO43 - UART RX: IO44 - Status LED (orange): IO16 - Status LED (blue) I015 Interrupts - IMU Interrupt: IO48 - Fuel Gauge Interrupt: IO17 - Touch Interrupt 1: IO4 - Touch Interrupt 2: IO5 - Touch Interrupt 3: IO6 - Touch Interrupt 4: IO7"
- note removed: "D"
- note removed: "G"
- note removed: "GPIO/SPI CONNECTOR"
- note removed: "I2C Level Shifting"
- note removed: "I2C OUT"
- note removed: "LIPO/LI-ION CONNECTOR"
- note removed: "S"
- note removed: "STATUS LED"
- note removed: "Touch Board Interrupt Pins - EVT1: IO7 - EVT2: IO6 - EVT3: IO5 - EVT4: IO4"
- moved on the sheet: BT1, BT2, C10, C11, C12, C13, C15, C19, C4, C5, C6, C7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

Commit message: switch back to revision 2 design
Parts:
- removed C16, C17, C20: 1uF, Capacitor_SMD:C_0402_1005Metric, symbol Device:C
- removed C18, C21: 0.1uF, Capacitor_SMD:C_0402_1005Metric, symbol Device:C
- removed SYS4: SYS, symbol power-symbols:VSYS
- removed U5: NCP167AMX330TBG, XDFN4_1X1_711AJ_ONS, symbol NCP167AMX330TBG:NCP167AMX330TBG
- removed U7: max3378eetd+t, 21-0137I_T1433-2_MXM, symbol MAX3378E:max3378eetd+t
- added Q1, Q2, Q3: BSS138, Package_TO_SOT_SMD:SOT-23, symbol Transistor_FET:BSS138
- added R14, R15, R21, R23: 2k2, Resistor_SMD:R_0402_1005Metric, symbol Device:R_US
- R22: value 2k -> 1k; Description Value Pkg 2 kOhms ±1% 0.1W, 1/10W Chip Resistor 0402 (1005 Metric) Au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 -> 1 kOhms ±1% 0.1W, 1/10W Chip Resistor 0402 (1005 Metric) Au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
- R24: value 470 -> 1k; Description Value Pkg 470 Ohms ±1% 0.1W, 1/10W Chip Resistor 0402 (1005 Metric) A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 -> 1 kOhms ±1% 0.1W, 1/10W Chip Resistor 0402 (1005 Metric) Au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; Mfg Part # ERJ-2RKF4700X -> ERJ-2RKF1001X
- R3: value 2k -> 1k; Description Value Pkg 2 kOhms ±1% 0.1W, 1/10W Chip Resistor 0402 (1005 Metric) Au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 -> 1 kOhms ±1% 0.1W, 1/10W Chip Resistor 0402 (1005 Metric) Au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; Mfg Part # ERJ-2RKF2001X -> ERJ-2RKF1001X
Connections:
- net +3V3_AUX is gone; now on net +3V3: TOUCH1.2 (Pin_2)
- net CIPO_1V8 is gone; now on net GND: IMU1.9 (SDO/AD0)
- net CS_1V8 is gone; now on net +1V8: IMU1.22 (~{CS})
- net +1V8: now also Q1.1 (G), Q2.1 (G), Q3.1 (G), R14.2, R15.2, R21.2
- net +3V3: now also R23.2
- net SCL: now also Q1.3 (D)
- net SDA: now also Q2.3 (D)
- net SYS: now also U4.3 (EN)
- net IMU_INT: now reaches IMU1.12 (INT1)
- net IMU_INT: now also Q3.2 (S), R21.1
- net CIPO_AUX renamed IO40
- net CLK_1V8 renamed LV_SCL
- net LV_SCL: now also Q1.2 (S), R14.1
- net CLK_AUX renamed IO42
- net COPI_1V8 renamed LV_SDA
- net LV_SDA: now also Q2.2 (S), R15.1
- net COPI_AUX renamed IO39
- net CS_AUX renamed IO41
- net LDO_EN renamed IO48
- net IO48: now also Q3.3 (D), R23.1; no longer U4.3 (EN)
- no-connect marks 10 -> 9
Other:
- note added: "3.3V Regulator"
- note added: "4 pin JST-SH connector to daisy chain touch board interrupts, alternatively can connect to the SPI2 controller on ESP32-S3"
- note added: "CHARGER CONFIGURATION"
- note added: "CHARGING STATUS LEDS"
- note added: "Charge Limit 2kOhm = 500mA"
- note added: "Charge Termincation Current 24.9koHm = 40mA charge termination"
- note added: "Comms - SDA: IO21 - SCL: IO14 - USBD+: IO20 - USBD-: IO19 - COPI: 10 - CIPO: 13 - SCLK: 12 - CS0: 11 Peripherals - FSR: IO8 - Button: IO9 - UART TX: IO43 - UART RX: IO44 - Status LED (orange): IO16 - Status LED (blue) I015 Interrupts - IMU Interrupt: IO48 - Fuel Gauge Interrupt: IO17 - Touch Interrupt 1: IO4 - Touch Interrupt 2: IO5 - Touch Interrupt 3: IO6 - Touch Interrupt 4: IO7"
- note added: "D"
- note added: "G"
- note added: "GPIO/SPI CONNECTOR"
- note added: "I2C Level Shifting"
- note added: "I2C OUT"
- note added: "LIPO/LI-ION CONNECTOR"
- note added: "S"
- note added: "STATUS LED"
- note added: "Touch Board Interrupt Pins - EVT1: IO7 - EVT2: IO6 - EVT3: IO5 - EVT4: IO4"
- note removed: "CHARGER CONFIG"
- note removed: "Charge Termination Current 24.9koHm = 40mA charge termination"
- note removed: "Charge resistor 1k = 1000mA 2k = 500mA 5k = 100mA"
- note removed: "Comms - USBD+: IO20 - USBD-: IO19 - UART TX: IO43 - UART RX: IO44 I2C - SDA: IO21 - SCL: IO14 SPI - COPI: 10 - CIPO: 13 - SCLK: 12 - CS0: 11 - COPI_AUX: 39 - CIPO_AUX: 40 - CLK_AUX: 42 - CS_AUX: 41 Peripherals - LDO ENABLE: 48 - FSR: IO8 - Button: IO9 - Status LED (orange): IO16 - Status LED (blue) I015 Interrupts - Fuel Gauge Interrupt: IO17"
- note removed: "ESD Protection IC"
- note removed: "GPIO CONNECTORS"
- note removed: "LIPO/LI-ION"
- note removed: "Main 3.3V Regulator"
- note removed: "Peripheral 3.3V Regulator"
- note removed: "STATUS LEDS"
- moved on the sheet: BT1, BT2, C10, C11, C12, C13, C15, C19, C4, C5, C6, C7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
