File: hardware/PCB/enchantiS3-board/enchantiS3.kicad_sch (KiCad schematic)
At the start: 71 parts, among them J1 USB_C_Receptacle_USB2.0, Q1 BSS138, Q2 BSS138, Q3 BSS138, SW1 B3U-1000P, SW2 B3U-1000P, U1 USBLC6-2P6, U2 MCP73871, U3 NCP167AMX330TBG, U4 NCP167AMX180TBG

Commit message: simplify rev3 design to only add an extra regulator
Parts:
- added C16, C17: 1uF, Capacitor_SMD:C_0402_1005Metric, symbol Device:C
- added SYS4: SYS, symbol power-symbols:VSYS
- added U5: NCP167AMX330TBG, XDFN4_1X1_711AJ_ONS, symbol NCP167AMX330TBG:NCP167AMX330TBG
Connections:
- net +3V3: no longer TOUCH1.2 (Pin_2)
- net GND: now also C16.2, C17.2, U5.2 (GND), U5.5 (GND)
- net IO39: now also U5.3 (EN)
- net SYS: now also C17.1, SYS4.1 (SYS), U5.4 (IN)
- new net 3V3_AUX: C16.1, TOUCH1.2 (Pin_2), U5.1 (OUT)
Other:
- note added: "3.3V - AUX Regulator"
- note removed: "CHARGING STATUS LEDS"
- moved on the sheet: C11, C12, C4, C5, R10, R22, R24, R3, R8, STATLED1, STATLED2, U3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

Commit message: updated enchantis3 board files, slowed down I2C clock
Parts:
- removed BT2: JST-PH-1x02-2.000mm, Connector_JST:JST_PH_S2B-PH-SM4-TB_1x02-1MP_P2.00mm_Horizontal, symbol Connector_Generic_MountingPin:Conn_01x02_MountingPin
Other:
- note removed: "Pads, to solder for battery connector on the botttom of board"
Changed lines of the file:
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@@
     (stroke (width 0) (type default))
   )
-  (wire (pts (xy 165.1 257.81) (xy 165.1 270.51))
-    (stroke (width 0) (type default))
-  )
   (wire (pts (xy 402.59 128.27) (xy 379.73 128.27))
     (stroke (width 0) (type default))
@@
     (stroke (width 0) (type default))
   )
-  (wire (pts (xy 165.1 250.19) (xy 165.1 255.27))
-    (stroke (width 0) (type default))
-  )
   (wire (pts (xy 350.52 130.81) (xy 355.6 130.81))
     (stroke (width 0) (type default))
@@
     (stroke (width 0) (type default))
   )
-  (wire (pts (xy 170.18 266.7) (xy 170.18 262.89))
-    (stroke (width 0) (type default))
-  )
   (wire (pts (xy 374.65 214.63) (xy 381 214.63))
     (stroke (width 0) (type default))
@@
     (effects (font (size 4 4) (color 0 0 0 1)) (justify left bottom))
   )
-  (text "Pads, to solder for battery connector \non the botttom of board"
-    (at 149.86 281.94 0)
-    (effects (font (size 1.27 1.27)) (justify left bottom))
-  )
   (text "STATUS LED" (at 281.94 119.38 0)
     (effects (font (size 4 4) (color 0 0 0 1)) (justify left bottom))
@@
     )
   )
-  (symbol (lib_id "Connector_Generic_MountingPin:Conn_01x02_MountingPin") (at 170.18 255.27 0) (unit 1)
-    (in_bom no) (on_board yes) (dnp no) (fields_autoplaced)
-    (property "Reference" "BT2" (at 173.99 253.6189 0)
-      (effects (font (size 1.27 1.27)) (justify left))
-    )
-    (property "Value" "JST-PH-1x02-2.000mm" (at 173.99 256.1589 0)
-      (effects (font (size 1.27 1.27)) (justify left) hide)
-    )
-    (property "Footprint" "Connector_JST:JST_PH_S2B-PH-SM4-TB_1x02-1MP_P2.00mm_Horizontal" (at 170.18 255.27 0)
-      (effects (font (size 1.27 1.27)) hide)
-    )
-    (property "Datasheet" "https://www.jst-mfg.com/product/pdf/eng/ePH.pdf" (at 170.18 255.27 0)
-      (effects (font (size 1.27 1.27)) hide)
-    )
-    (property "Description Value Pkg" "Connector Header Surface Mount, Right Angle 2 position 0.079\" (2.00mm)" (at 170.18 255.27 0)
-      (effects (font (size 1.27 1.27)) hide)
-    )
-    (property "Mfg Part #" "S2B-PH-SM4-TB" (at 170.18 255.27 0)
-      (effects (font (size 1.27 1.27)) hide)
-    )
-    (property "Manufacturer" "JST Sales America Inc." (at 170.18 255.27 0)
-      (effects (font (size 1.27 1.27)) hide)
-    )
-    (property "mpn" "B2B-PH-SM4-TBT" (at 170.18 255.27 0)
-      (effects (font (size 1.27 1.27)) hide)
-    )
-    (pin "1")
-    (pin "2")
-    (pin "MP")
-    (instances
-      (project "enchantiS3"
-        (path "/1e57a4ff-0c95-4e2b-9e56-d9bf8e99c9a1"
-          (reference "BT2") (unit 1)
-        )
-      )
-      (project "tstick_pcb"
-        (path "/ecdbf224-0069-4dc3-a7df-492909ab59c7"
-          (reference "BT1") (unit 1)
-        )
-      )
-    )
-  )
   (symbol (lib_id "power:+1V8") (at 293.37 86.36 0) (unit 1)
     (in_bom yes) (on_board yes) (dnp no) (fields_autoplaced)
@@
     )
   )
-  (symbol (lib_id "power:+BATT") (at 165.1 250.19 0) (unit 1)
-    (in_bom yes) (on_board yes) (dnp no) (fields_autoplaced)
-    (property "Reference" "#PWR062" (at 165.1 254 0)
-      (effects (font (size 1.27 1.27)) hide)
-    )
-    (property "Value" "+BATT" (at 165.1 245.11 0)
-      (effects (font (size 1.27 1.27)))
-    )
-    (property "Footprint" "" (at 165.1 250.19 0)
-      (effects (font (size 1.27 1.27)) hide)
-    )
-    (property "Datasheet" "" (at 165.1 250.19 0)
-      (effects (font (size 1.27 1.27)) hide)
-    )
-    (pin "1")
-    (instances
-      (project "enchantiS3"
-        (path "/1e57a4ff-0c95-4e2b-9e56-d9bf8e99c9a1"
-          (reference "#PWR062") (unit 1)
-        )
-      )
-      (project "tstick_pcb"
-        (path "/ecdbf224-0069-4dc3-a7df-492909ab59c7"
-          (reference "#PWR029") (unit 1)
-        )
-      )
-    )
-  )
   (symbol (lib_name "GND_1") (lib_id "power:GND") (at 345.44 153.67 0) (unit 1)
     (in_bom yes) (on_board yes) (dnp no) (fields_autoplaced)
@@
     )
   )
-  (symbol (lib_name "GND_1") (lib_id "power:GND") (at 170.18 266.7 0) (unit 1)
-    (in_bom yes) (on_board yes) (dnp no) (fields_autoplaced)
-    (property "Reference" "#PWR075" (at 170.18 273.05 0)
-      (effects (font (size 1.27 1.27)) hide)
-    )
-    (property "Value" "GND" (at 170.18 271.78 0)
-      (effects (font (size 1.27 1.27)))
-    )
-    (property "Footprint" "" (at 170.18 266.7 0)
-      (effects (font (size 1.27 1.27)) hide)
-    )
-    (property "Datasheet" "" (at 170.18 266.7 0)
-      (effects (font (size 1.27 1.27)) hide)
-    )
-    (pin "1")
-    (instances
-      (project "enchantiS3"
-        (path "/1e57a4ff-0c95-4e2b-9e56-d9bf8e99c9a1"
-          (reference "#PWR075") (unit 1)
-        )
-      )
-      (project "tstick_pcb"
-        (path "/ecdbf224-0069-4dc3-a7df-492909ab59c7"
-          (reference "#PWR010") (unit 1)
-        )
-      )
-    )
-  )
   (symbol (lib_name "GND_2") (lib_id "power:GND") (at 121.92 48.26 0) (unit 1)
     (in_bom yes) (on_board yes) (dnp no) (fields_autoplaced)
@@
         )
       )
-    )
-  )
-  (symbol (lib_id "power:-BATT") (at 165.1 270.51 180) (unit 1)
-    (in_bom yes) (on_board yes) (dnp no) (fields_autoplaced)
-    (property "Reference" "#PWR064" (at 165.1 266.7 0)
-      (effects (font (size 1.27 1.27)) hide)
-    )
-    (property "Value" "-BATT" (at 165.1 275.59 0)
-      (effects (font (size 1.27 1.27)))
-    )
-    (property "Footprint" "" (at 165.1 270.51 0)
-      (effects (font (size 1.27 1.27)) hide)
-    )
-    (property "Datasheet" "" (at 165.1 270.51 0)
-      (effects (font (size 1.27 1.27)) hide)
-    )
-    (pin "1")
-    (instances
-      (project "enchantiS3"
-        (path "/1e57a4ff-0c95-4e2b-9e56-d9bf8e99c9a1"
-          (reference "#PWR064") (unit 1)
-        )
-      )
-      (project "tstick_pcb"
-        (path "/ecdbf224-0069-4dc3-a7df-492909ab59c7"
-          (reference "#PWR03") (unit 1)
-        )
-      )
